File: PCB/WLS3/WLS3/WLS3.kicad_sch (KiCad schematic)
At the start: 38 parts, among them J1 Sensor, J10 Sensor, J11 OLED Display, J12 Battery, J13 PushButton, J2 Sensor Wire, Q10 IRF9540N, Q11 BC547, SW10 CAL DRY, SW11 CAL WET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

Commit message: Updated PCB sensor
Parts:
- added H1, H2, H3, H4: MountingHole, MountingHole:MountingHole_3.2mm_M3, symbol Mechanical:MountingHole
- added R4: 10E, Resistor_THT:R_Axial_DIN0207_L6.3mm_D2.5mm_P10.16mm_Horizontal, symbol Device:R_Small
- C13, C2, C3: footprint Capacitor_THT:CP_Radial_D10.0mm_P5.00mm -> Capacitor_THT:CP_Radial_D8.0mm_P5.00mm
- renumbered J2 to J5
Connections:
- net +5VA: now also R4.1; no longer U1.4 (R)
- net GNDA: now also J1.3 (Pin_3); no longer J1.1 (Pin_1)
- net at D1.2 (A): now also J1.1 (Pin_1); no longer J1.3 (Pin_3)
- new net: R4.2, U1.4 (R)
Other:
- moved on the sheet: R3
